Commit message: upgrades the camera

File: catkin_ws/src/my_robot/urdf/my_robot.xacro (robot description, xacro)
@@ -207,4 +207,11 @@
         <material>Gazebo/Green</material>
     </gazebo> -->
+    <joint name="camera_optical_joint" type="fixed">
+        <origin xyz="0 0 0" rpy="-1.5707 0 -1.5707"/>
+        <parent link="camera"/>
+        <child link="camera_link_optical"/>
+    </joint>
+    <link name="camera_link_optical">
+    </link>
     <joint name="camera_joint" type="fixed">
         <origin xyz="0.2 0 0" rpy="0 0 0"/>
